File: psu/pm1000_psu/pm1000_psu.kicad_sch (KiCad schematic)
At the start: 42 parts, among them J3 Screw_Terminal_01x05, U1 LM317_TO-220, U2 LM317_TO-220, U3 LM317_TO-220

Commit message: set led resistors to 22k, place new psu terminal block
Parts:
- J3: footprint (none) -> TerminalBlock_Phoenix:TerminalBlock_Phoenix_PT-1,5-5-5.0-H_1x05_P5.00mm_Horizontal
- R10, R11, R12, R2: value 2k2 -> 22k
Changed lines of the file:
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@@
 			)
 		)
-		(property "Value" "2k2"
+		(property "Value" "22k"
 			(at 76.2 168.9099 0)
 			(effects
@@
 			)
 		)
-		(property "Value" "2k2"
+		(property "Value" "22k"
 			(at 60.96 168.9099 0)
 			(effects
@@
 			)
 		)
-		(property "Value" "2k2"
+		(property "Value" "22k"
 			(at 233.68 36.83 90)
 			(effects
@@
 			)
 		)
-		(property "Footprint" ""
+		(property "Footprint" "TerminalBlock_Phoenix:TerminalBlock_Phoenix_PT-1,5-5-5.0-H_1x05_P5.00mm_Horizontal"
 			(at 38.1 46.99 0)
 			(effects
@@
 			)
 		)
-		(property "Value" "2k2"
+		(property "Value" "22k"
 			(at 45.72 168.9099 0)
 			(effects
