File: pm1000_psu/pm1000_psu.kicad_pcb (KiCad board)
At the start: 2 copper layers, 105 x 35 mm, 42 parts, among them J3 Screw_Terminal_01x05, U1 LM317_TO-220, U2 LM317_TO-220, U3 LM317_TO-220

Commit message: clean up project structure, organize psu silkscreen
Parts:
- renumbered C5 to C3, C3 to C4, C4 to C5, C8 to C6, C9 to C7, C6 to C8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
Routing:
- net +48V: track 57.2 -> 60.2 mm
- net Net-(U3-ADJ): track 34.1 -> 31.3 mm
Other:
- board size 105 x 35 mm -> 107 x 37 mm
- board text added: "${REFERENCE}"
