File: pm1000_psu/pm1000_psu.kicad_pcb (KiCad board)
At the start: 2 copper layers, 107 x 37 mm, 42 parts, among them J1 Screw_Terminal_01x05, U1 LM317_TO-220, U2 LM317_TO-220, U3 LM317_TO-220

Commit message: re-engineer psu board
Parts:
- removed R10, R11, R12, R9: 22k, Resistor_THT:R_Axial_DIN0207_L6.3mm_D2.5mm_P10.16mm_Horizontal
- removed R8: 7k5, Resistor_THT:R_Axial_DIN0207_L6.3mm_D2.5mm_P10.16mm_Horizontal
- removed RV1, RV2, RV3: 2k, Potentiometer_THT:Potentiometer_Piher_PT-10-V05_Vertical
- removed U3: LM317_TO-220, Package_TO_SOT_THT:TO-220-3_Vertical
- added C10: 22uF 63V, Capacitor_THT:CP_Radial_D8.0mm_P3.50mm, F.Cu at (102.5, 50.8)
- C1: value 220uF 80V -> 2200uF 80V; footprint Capacitor_THT:CP_Radial_D12.5mm_P5.00mm -> Capacitor_THT:CP_Radial_D22.0mm_P10.00mm_SnapIn
- C2: value 10uF 80V -> 2200uF 80V; footprint Capacitor_THT:CP_Radial_D6.3mm_P2.50mm -> Capacitor_THT:CP_Radial_D22.0mm_P10.00mm_SnapIn
- C3, C4, C6, C8: value 10uF 80V -> 100n; footprint Capacitor_THT:CP_Radial_D6.3mm_P2.50mm -> Capacitor_THT:C_Disc_D5.0mm_W2.5mm_P2.50mm
- C5, C7, C9: value 100n -> 22uF 63V; footprint Capacitor_THT:C_Disc_D5.0mm_W2.5mm_P2.50mm -> Capacitor_THT:CP_Radial_D8.0mm_P3.50mm
- D1, D2, D5, D6, D7: value 1n4004 -> D_Small
- D10, D8, D9: value LED_Small -> D_Small; footprint LED_THT:LED_D3.0mm -> Diode_THT:D_DO-41_SOD81_P10.16mm_Horizontal
- D3, D4: value 1n4004 -> LED_Small; footprint Diode_THT:D_DO-41_SOD81_P10.16mm_Horizontal -> LED_THT:LED_D3.0mm
- J1: value Screw_Terminal_01x05 -> Power Led; footprint TerminalBlock_Phoenix:TerminalBlock_Phoenix_PT-1,5-5-5.0-H_1x05_P5.00mm_Horizontal -> Connector_Molex:Molex_KK-254_AE-6410-02A_1x02_P2.54mm_Vertical
- J2: value ~ -> Screw_Terminal_01x05; footprint Connector_Molex:Molex_KK-396_5273-02A_1x02_P3.96mm_Vertical -> TerminalBlock_Phoenix:TerminalBlock_Phoenix_PT-1,5-5-5.0-H_1x05_P5.00mm_Horizontal
- J3: value ~ -> Channel 1
- J4: value ~ -> Phantom
- J5: value ~ -> Channel 2; footprint Connector_Molex:Molex_KK-254_AE-6410-02A_1x02_P2.54mm_Vertical -> Connector_Molex:Molex_KK-396_5273-02A_1x02_P3.96mm_Vertical
- R1, R2: value 100R 1W -> 22k; footprint Resistor_THT:R_Axial_DIN0411_L9.9mm_D3.6mm_P15.24mm_Horizontal -> Resistor_THT:R_Axial_DIN0207_L6.3mm_D2.5mm_P10.16mm_Horizontal
- R3: value 240r -> 22k
- moved J1 93.4 mm to (115.0, 62.5), turned to 0 degrees
- moved D3 74.7 mm to (101.7, 32.0)
- moved C4 72.4 mm to (119.0, 31.5), turned to -90 degrees
- moved R1 61.1 mm to (121.5, 58.1), turned to 90 degrees
- moved D6 59.6 mm to (31.3, 64.0), turned to 0 degrees
- moved D4 54.4 mm to (77.0, 32.0)
- moved R6 53.9 mm to (108.0, 35.3), turned to -90 degrees
- moved C5 40.6 mm to (90.0, 51.0), turned to -90 degrees
- moved C7 39.3 mm to (115.5, 50.5), turned to -90 degrees
- moved J5 39.0 mm to (92.0, 64.0), turned to 90 degrees
- moved D9 38.4 mm to (86.5, 46.2), turned to 90 degrees
- moved D10 37.0 mm to (111.5, 45.8), turned to 90 degrees
- moved U1 36.9 mm to (83.9, 32.5), turned to 0 degrees
- moved U2 35.8 mm to (109.0, 32.5), turned to 0 degrees
- moved D5 32.6 mm to (31.3, 60.5), turned to 0 degrees
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Connections:
- C2 pad 1: Net-(D5-K) -> unreg
- C3 pad 1: Net-(D6-K) -> unreg
- C4 pad 1: +44V A -> unreg
- C5 pad 1: +44V A -> +44V
- C6 pad 1: +44V B -> +44V
- C7 pad 1: +44V B -> +Phantom
- C8 pad 1: +48V -> +Phantom
- C9 pad 1: +48V -> Net-(D9-A)
- D10 pad 1: Net-(D10-K) -> +Phantom
- D10 pad 2: +44V B -> Net-(D10-A)
- D3 pad 1: Net-(D1-A) -> Net-(D3-K)
- D3 pad 2: GND -> +Phantom
- D4 pad 1: Net-(D2-A) -> Net-(D4-K)
- D4 pad 2: GND -> +44V
- D5 pad 1: Net-(D5-K) -> Net-(D1-A)
- D5 pad 2: +44V A -> GND
- D6 pad 1: Net-(D6-K) -> Net-(D2-A)
- D6 pad 2: +44V B -> GND
- D7 pad 2: +48V -> +44V
- D8 pad 1: Net-(D8-K) -> unreg
- D8 pad 2: +48V -> +Phantom
- D9 pad 1: Net-(D9-K) -> +44V
- D9 pad 2: +44V A -> Net-(D9-A)
- J1 pad 1: Net-(D2-A) -> GND
- J2 pad 1: GND -> Net-(D2-A)
- J2 pad 2: +44V A -> Net-(J2-Pin_2)
- J3 pad 2: +44V B -> +44V
- J4 pad 2: +48V -> +Phantom
- J5 pad 2: Net-(J5-Pin_2) -> +44V
- R1 pad 1: unreg -> Net-(J1-Pin_2)
- R1 pad 2: Net-(D5-K) -> +Phantom
- R2 pad 1: unreg -> GND
- R2 pad 2: Net-(D6-K) -> Net-(D3-K)
- R3 pad 1: Net-(U1-ADJ) -> GND
- R3 pad 2: +44V A -> Net-(D4-K)
- R4 pad 1: Net-(U2-ADJ) -> Net-(D9-A)
- R4 pad 2: +44V B -> +44V
- R5 pad 1: Net-(U3-ADJ) -> Net-(D10-A)
- R5 pad 2: +48V -> +Phantom
- R6 pad 1: GND -> Net-(D10-A)
- R6 pad 2: Net-(R6-Pad2) -> GND
- R7 pad 1: GND -> Net-(D9-A)
- R7 pad 2: Net-(R7-Pad2) -> GND
- U1 pad 1: Net-(U1-ADJ) -> Net-(D9-A)
- U1 pad 2: +44V A -> +44V
- U1 pad 3: Net-(D5-K) -> unreg
- U2 pad 1: Net-(U2-ADJ) -> Net-(D10-A)
- U2 pad 2: +44V B -> +Phantom
- U2 pad 3: Net-(D6-K) -> unreg
Routing:
- net +44V: track 0.00 -> 65.1 mm
- net +Phantom: track 0.00 -> 63.1 mm
- net +48V: track 60.2 -> 0.00 mm
- net +44V B: track 47.0 -> 0.00 mm
- net +44V A: track 46.8 -> 0.00 mm
- net Net-(U3-ADJ): track 31.3 -> 0.00 mm
- net Net-(U2-ADJ): track 30.0 -> 0.00 mm
- net Net-(U1-ADJ): track 29.9 -> 0.00 mm
- net Net-(D9-A): track 0.00 -> 28.0 mm
- net Net-(D5-K): track 26.6 -> 0.00 mm
- net Net-(D6-K): track 26.3 -> 0.00 mm
- net Net-(D10-A): track 0.00 -> 26.1 mm
- net Net-(D1-A): track 11.7 -> 36.0 mm
- net unreg: track 119.2 -> 105.7 mm
- net Net-(J5-Pin_2): track 11.2 -> 0.00 mm
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Other:
- board text removed: "${REFERENCE}"

Commit message: finish psu layout
Parts:
- removed D3: LED_Small, LED_THT:LED_D3.0mm
- removed R2: 22k, Resistor_THT:R_Axial_DIN0207_L6.3mm_D2.5mm_P10.16mm_Horizontal
- added C11: 22uF 63V, Capacitor_THT:CP_Radial_D8.0mm_P3.50mm, F.Cu at (72.5, 50.0)
- added C12: 100n, Capacitor_THT:C_Disc_D5.0mm_W2.5mm_P2.50mm, F.Cu at (63.5, 58.8)
- added C13: 22uF 63V, Capacitor_THT:CP_Radial_D8.0mm_P3.50mm, F.Cu at (63.5, 50.0)
- added C14: 2200uF 80V, Capacitor_THT:CP_Radial_D22.0mm_P10.00mm_SnapIn, F.Cu at (48.0, 54.0)
- added D11: D_Small, Diode_THT:D_DO-41_SOD81_P10.16mm_Horizontal, F.Cu at (114.8, 40.5)
- added D12: D_Small, Diode_THT:D_DO-41_SOD81_P10.16mm_Horizontal, F.Cu at (62.5, 33.4)
- added D13: D_Small, Diode_THT:D_DO-41_SOD81_P10.16mm_Horizontal, F.Cu at (72.6, 40.4)
- added R10: 8k2, Resistor_THT:R_Axial_DIN0207_L6.3mm_D2.5mm_P10.16mm_Horizontal, F.Cu at (62.4, 43.9)
- added R8: 8k2, Resistor_THT:R_Axial_DIN0207_L6.3mm_D2.5mm_P10.16mm_Horizontal, F.Cu at (104.8, 44.0)
- added R9: 240r, Resistor_THT:R_Axial_DIN0207_L6.3mm_D2.5mm_P10.16mm_Horizontal, F.Cu at (62.5, 36.9)
- added U3: LM317_TO-220, Package_TO_SOT_THT:TO-220-3_Vertical, F.Cu at (69.5, 29.9)
- C10, C5, C7: value 22uF 63V -> 100n; footprint Capacitor_THT:CP_Radial_D8.0mm_P3.50mm -> Capacitor_THT:C_Disc_D5.0mm_W2.5mm_P2.50mm
- C2: value 2200uF 80V -> 100n; footprint Capacitor_THT:CP_Radial_D22.0mm_P10.00mm_SnapIn -> Capacitor_THT:C_Disc_D5.0mm_W2.5mm_P2.50mm
- C4, C6, C8: value 100n -> 22uF 63V; footprint Capacitor_THT:C_Disc_D5.0mm_W2.5mm_P2.50mm -> Capacitor_THT:CP_Radial_D8.0mm_P3.50mm
- D5: value D_Small -> LED_Small; footprint Diode_THT:D_DO-41_SOD81_P10.16mm_Horizontal -> LED_THT:LED_D3.0mm
- J1: value Power Led -> Screw_Terminal_01x05; footprint Connector_Molex:Molex_KK-254_AE-6410-02A_1x02_P2.54mm_Vertical -> TerminalBlock_Phoenix:TerminalBlock_Phoenix_PT-1,5-5-5.0-H_1x05_P5.00mm_Horizontal
- J2: value Screw_Terminal_01x05 -> Power Led; footprint TerminalBlock_Phoenix:TerminalBlock_Phoenix_PT-1,5-5-5.0-H_1x05_P5.00mm_Horizontal -> Connector_Molex:Molex_KK-254_AE-6410-02A_1x02_P2.54mm_Vertical
- J3: value Channel 1 -> Output A
- J4: value Phantom -> Output B; footprint Connector_Molex:Molex_KK-254_AE-6410-02A_1x02_P2.54mm_Vertical -> Connector_Molex:Molex_KK-396_5273-02A_1x02_P3.96mm_Vertical
- J5: value Channel 2 -> Phantom; footprint Connector_Molex:Molex_KK-396_5273-02A_1x02_P3.96mm_Vertical -> Connector_Molex:Molex_KK-254_AE-6410-02A_1x02_P2.54mm_Vertical
- R4: value 240r -> 22k
- R6: value 7k5 -> 240r
- R7: value 7k5 -> 8k2
- moved J1 91.6 mm to (23.5, 57.5), turned to 90 degrees
- moved D5 77.9 mm to (109.0, 66.5), turned to 90 degrees
- moved D7 60.9 mm to (31.0, 49.0)
- moved J2 51.1 mm to (74.0, 65.0), turned to 180 degrees
- moved R1 45.0 mm to (76.6, 56.0), turned to 180 degrees
- moved C10 42.9 mm to (65.0, 29.9), turned to 180 degrees
- moved D4 36.2 mm to (88.0, 66.5), turned to 90 degrees
- moved R4 33.0 mm to (105.0, 56.5)
- moved D8 32.0 mm to (83.6, 33.5), turned to 0 degrees
- moved C6 31.3 mm to (114.8, 50.0), turned to 0 degrees
- moved C4 31.1 mm to (94.0, 50.0), turned to 0 degrees
- moved C9 28.7 mm to (105.7, 50.0), turned to 0 degrees
- moved J5 24.5 mm to (67.5, 65.0), turned to 180 degrees
- moved C8 24.1 mm to (84.9, 50.0), turned to 0 degrees
- moved C2 23.9 mm to (86.2, 30.0), turned to 180 degrees
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Connections:
- C10 pad 1: Net-(D10-A) -> unreg
- C4 pad 1: unreg -> +44VA
- C5 pad 1: +44V -> +44VA
- C6 pad 1: +44V -> +44VB
- C7 pad 1: +Phantom -> +44VB
- C8 pad 1: +Phantom -> Net-(D10-A)
- C9 pad 1: Net-(D9-A) -> Net-(D11-A)
- D10 pad 1: +Phantom -> +44VA
- D4 pad 2: +44V -> +44VA
- D5 pad 1: Net-(D1-A) -> Net-(D5-K)
- D5 pad 2: GND -> +44VB
- D6 pad 1: Net-(D2-A) -> Net-(D1-A)
- D7 pad 1: unreg -> Net-(D2-A)
- D7 pad 2: +44V -> GND
- D8 pad 2: +Phantom -> +44VA
- D9 pad 1: +44V -> unreg
- D9 pad 2: Net-(D9-A) -> +44VB
- J1 pad 1: GND -> Net-(D2-A)
- J2 pad 1: Net-(D2-A) -> GND
- J3 pad 2: +44V -> +44VA
- J4 pad 2: +Phantom -> +44VB
- J5 pad 2: +44V -> +Phantom
- R1 pad 1: Net-(J1-Pin_2) -> Net-(J2-Pin_2)
- R4 pad 1: Net-(D9-A) -> GND
- R4 pad 2: +44V -> Net-(D5-K)
- R5 pad 2: +Phantom -> +44VA
- R6 pad 1: Net-(D10-A) -> Net-(D11-A)
- R6 pad 2: GND -> +44VB
- R7 pad 1: Net-(D9-A) -> Net-(D10-A)
- U1 pad 1: Net-(D9-A) -> Net-(D10-A)
- U1 pad 2: +44V -> +44VA
- U2 pad 1: Net-(D10-A) -> Net-(D11-A)
- U2 pad 2: +Phantom -> +44VB
Routing:
- net +44V: track 65.1 -> 0.00 mm
- net +44VA: track 0.00 -> 43.3 mm
- net +44VB: track 0.00 -> 37.8 mm
- net Net-(D9-A): track 28.0 -> 0.00 mm
- net unreg: track 105.7 -> 133.1 mm
- net Net-(D13-A): track 0.00 -> 23.5 mm
- net Net-(D11-A): track 0.00 -> 23.3 mm
- net Net-(D2-A): track 36.8 -> 14.5 mm
- net +Phantom: track 63.1 -> 41.1 mm
- net Net-(D1-A): track 36.0 -> 15.3 mm
- net Net-(J2-Pin_2): track 5.00 -> 11.1 mm
- net Net-(D5-K): track 0.00 -> 4.07 mm
- net Net-(D3-K): track 3.64 -> 0.00 mm
- net Net-(D10-A): track 26.1 -> 23.5 mm
- net Net-(J1-Pin_2): track 6.06 -> 5.00 mm
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Other:
- board size 107 x 37 mm -> 107 x 42 mm
