File: pm1000_psu/pm1000_psu.kicad_sch (KiCad schematic)
At the start: 42 parts, among them J3 Screw_Terminal_01x05, U1 LM317_TO-220, U2 LM317_TO-220, U3 LM317_TO-220

Commit message: clean up project structure, organize psu silkscreen
Parts:
- renumbered C5 to C3, C3 to C4, C4 to C5, C8 to C6, C9 to C7, C6 to C8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
Other:
- moved on the sheet: C1, C2, C3, C4, C5, C6, C7, C8, C9, D1, D10, D2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
