File: pm1000_phantom/pm1000_phantom.kicad_sch (KiCad schematic)
At the start: 17 parts, among them J1 2 pin 2,54mm Molex, J10 2 pin 2,54mm Molex, J2 2 pin 2,54mm Molex, J3 2 pin 2,54mm Molex, J4 2 pin 2,54mm Molex, J5 2 pin 2,54mm Molex, J6 3 pin 2,54mm Molex, J7 3 pin 2,54mm Molex, J8 3 pin 2,54mm Molex, J9 3 pin 2,54mm Molex

Commit message: fix phantom board labels
Parts:
- J1: value 2 pin 2,54mm Molex -> 48V in
- J2: value 2 pin 2,54mm Molex -> Switch A
- J3: value 2 pin 2,54mm Molex -> Switch B
- J4: value 2 pin 2,54mm Molex -> Led A
- J5: value 2 pin 2,54mm Molex -> Led B
Changed lines of the file:
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@@
 			)
 		)
-		(property "Value" "2 pin 2,54mm Molex"
-			(at 102.87 35.56 0)
-			(effects
-				(font
-					(size 1.27 1.27)
-				)
-				(justify left)
-				(hide yes)
+		(property "Value" "Led A"
+			(at 99.06 37.084 0)
+			(effects
+				(font
+					(size 1.27 1.27)
+				)
+				(justify left)
 			)
 		)
@@
 					(size 1.27 1.27)
 				)
+				(hide yes)
 			)
 		)
@@
 			)
 		)
-		(property "Value" "2 pin 2,54mm Molex"
-			(at 102.87 22.86 0)
-			(effects
-				(font
-					(size 1.27 1.27)
-				)
-				(justify left)
-				(hide yes)
+		(property "Value" "Switch A"
+			(at 98.806 24.13 0)
+			(effects
+				(font
+					(size 1.27 1.27)
+				)
+				(justify left)
 			)
 		)
@@
 					(size 1.27 1.27)
 				)
+				(hide yes)
 			)
 		)
@@
 			)
 		)
-		(property "Value" "2 pin 2,54mm Molex"
-			(at 41.91 27.94 0)
-			(effects
-				(font
-					(size 1.27 1.27)
-				)
-				(justify left)
-				(hide yes)
+		(property "Value" "48V in"
+			(at 39.116 29.21 0)
+			(effects
+				(font
+					(size 1.27 1.27)
+				)
+				(justify left)
 			)
 		)
@@
 					(size 1.27 1.27)
 				)
+				(hide yes)
 			)
 		)
@@
 			)
 		)
-		(property "Value" "2 pin 2,54mm Molex"
-			(at 170.18 35.56 0)
-			(effects
-				(font
-					(size 1.27 1.27)
-				)
-				(justify left)
-				(hide yes)
+		(property "Value" "Led B"
+			(at 165.862 36.576 0)
+			(effects
+				(font
+					(size 1.27 1.27)
+				)
+				(justify left)
 			)
 		)
@@
 					(size 1.27 1.27)
 				)
+				(hide yes)
 			)
 		)
@@
 			)
 		)
-		(property "Value" "2 pin 2,54mm Molex"
-			(at 170.18 22.86 0)
-			(effects
-				(font
-					(size 1.27 1.27)
-				)
-				(justify left)
-				(hide yes)
+		(property "Value" "Switch B"
+			(at 166.37 24.13 0)
+			(effects
+				(font
+					(size 1.27 1.27)
+				)
+				(justify left)
 			)
 		)
@@
 					(size 1.27 1.27)
 				)
-			)
-		)
+				(hide yes)
+			)
+		)

Commit message: phantom board connector descriptions
Parts:
- J10: value 2 pin 2,54mm Molex -> Power Led
- J6: value 3 pin 2,54mm Molex -> Mic A
- J7: value 3 pin 2,54mm Molex -> Mod A
- J8: value 3 pin 2,54mm Molex -> Mic B
- J9: value 3 pin 2,54mm Molex -> Mod B
Changed lines of the file:
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@@
 			)
 		)
-		(property "Value" "3 pin 2,54mm Molex"
+		(property "Value" "Mic B"
 			(at 133.35 74.93 0)
 			(effects
@@
 					(size 1.27 1.27)
 				)
-				(hide yes)
 			)
 		)
@@
 					(size 1.27 1.27)
 				)
+				(hide yes)
 			)
 		)
@@
 					(size 1.27 1.27)
 				)
+				(hide yes)
 			)
 		)
@@
 			)
 		)
-		(property "Value" "3 pin 2,54mm Molex"
+		(property "Value" "Mic A"
 			(at 35.56 74.93 0)
 			(effects
@@
 					(size 1.27 1.27)
 				)
-				(hide yes)
 			)
 		)
@@
 					(size 1.27 1.27)
 				)
+				(hide yes)
 			)
 		)
@@
 					(size 1.27 1.27)
 				)
+				(hide yes)
 			)
 		)
@@
 			)
 		)
-		(property "Value" "3 pin 2,54mm Molex"
-			(at 83.82 82.5499 0)
-			(effects
-				(font
-					(size 1.27 1.27)
-				)
-				(justify left)
-				(hide yes)
+		(property "Value" "Mod A"
+			(at 80.01 75.946 0)
+			(effects
+				(font
+					(size 1.27 1.27)
+				)
+				(justify left)
 			)
 		)
@@
 					(size 1.27 1.27)
 				)
+				(hide yes)
 			)
 		)
@@
 					(size 1.27 1.27)
 				)
+				(hide yes)
 			)
 		)
@@
 					(size 1.27 1.27)
 				)
+				(hide yes)
 			)
 		)
@@
 			)
 		)
-		(property "Value" "2 pin 2,54mm Molex"
+		(property "Value" "Power Led"
 			(at 50.8 111.76 0)
 			(effects
@@
 				)
 				(justify left)
-				(hide yes)
 			)
 		)
@@
 					(size 1.27 1.27)
 				)
+				(hide yes)
 			)
 		)
@@
 					(size 1.27 1.27)
 				)
+				(hide yes)
 			)
 		)
@@
 					(size 1.27 1.27)
 				)
+				(hide yes)
 			)
 		)
@@
 					(size 1.27 1.27)
 				)
+				(hide yes)
 			)
 		)
@@
 					(size 1.27 1.27)
 				)
+				(hide yes)
 			)
 		)
@@
 			)
 		)
-		(property "Value" "3 pin 2,54mm Molex"
-			(at 181.61 82.5499 0)
-			(effects
-				(font
-					(size 1.27 1.27)
-				)
-				(justify left)
-				(hide yes)
+		(property "Value" "Mod B"
+			(at 178.562 75.692 0)
+			(effects
+				(font
+					(size 1.27 1.27)
+				)
+				(justify left)
 			)
 		)
@@
 					(size 1.27 1.27)
 				)
+				(hide yes)
 			)
 		)
@@
 					(size 1.27 1.27)
 				)
+				(hide yes)
 			)
 		)
@@
 					(size 1.27 1.27)
 				)
-			)
-		)
+				(hide yes)
+			)
+		)
